File: RL78-flash-programmer.sch (KiCad schematic (older format))
At the start: 22 parts, among them J1 Conn_01x02, J2 USB_B, J3 Screw_Terminal_01x02, J4 Screw_Terminal_01x02, J8 Conn_02x05_Odd_Even, U1 74LS06, U2 74LS125, U3 FT232RL

Commit message: nc
Parts:
- U3: footprint prabhu:SSOP-28_5.3x10.2mm_P0.65mm -> Package_SO:SSOP-28_5.3x10.2mm_P0.65mm
Other:
- moved on the sheet: J1, J8
Changed lines of the file:
@@
 Sheet 1 1
 Title "RL78-flash-programmer"
-Date "2021-05-01"
+Date "2021-10-29"
 Rev "v1.2"
 Comp "PRABHU.YU@OUTLOOK.COM"
@@
 	8150 2300 8150 2200
 Wire Wire Line
-	2650 2100 2650 2850
+	2900 2100 2900 2850
 Wire Wire Line
 	4500 1750 4500 2150
@@
 F 0 "U3" H 6350 1700 50  0000 C CNN
 F 1 "FT232RL" H 6350 1600 50  0000 C CNN
-F 2 "prabhu:SSOP-28_5.3x10.2mm_P0.65mm" H 6350 400 50  0001 C CNN
+F 2 "Package_SO:SSOP-28_5.3x10.2mm_P0.65mm" H 6350 400 50  0001 C CNN
 F 3 "http://www.ftdichip.com/Products/ICs/FT232RL.htm" H 6350 650 50  0001 C CNN
 	1    5550 1400
@@
 Wire Wire Line
 	4750 2850 4400 2850
-Text Label 2500 2000 0    50   ~ 0
-TL
-Text Label 2500 2100 0    50   ~ 0
+Text Label 2750 2100 0    50   ~ 0
 RST
 Wire Wire Line
@@
 Wire Wire Line
 	7150 2750 8350 2750
-Text Notes 1650 2150 0    50   ~ 0
+Text Notes 2300 2150 0    50   ~ 0
 RST
-Text Notes 1700 2050 0    50   ~ 0
+Text Notes 2350 2050 0    50   ~ 0
 TL
-Text Notes 550  1800 0    50   ~ 0
+Text Notes 1250 1700 0    50   ~ 0
 GND
 Wire Wire Line
-	1450 2350 1450 2250
-Connection ~ 1450 2350
-Wire Wire Line
-	1250 2350 1450 2350
-Wire Wire Line
-	1450 2250 1450 2150
-Connection ~ 1450 2250
-Wire Wire Line
-	1250 2250 1450 2250
-Wire Wire Line
-	1450 2150 1450 2050
-Connection ~ 1450 2150
-Wire Wire Line
-	1250 2150 1450 2150
-Connection ~ 1450 2050
-Wire Wire Line
-	1450 2450 1450 2350
-Wire Wire Line
-	1250 2450 1450 2450
-Wire Wire Line
-	600  2450 600  2350
-Connection ~ 600  2450
-Wire Wire Line
-	750  2450 600  2450
-Wire Wire Line
-	600  2350 600  2250
-Connection ~ 600  2350
-Wire Wire Line
-	750  2350 600  2350
-Wire Wire Line
-	600  2250 600  2150
-Connection ~ 600  2250
-Wire Wire Line
-	750  2250 600  2250
-Wire Wire Line
-	600  2150 600  2050
-Connection ~ 600  2150
-Wire Wire Line
-	750  2150 600  2150
-Wire Wire Line
-	600  2050 750  2050
-Wire Wire Line
-	600  2750 600  2450
-Wire Wire Line
-	1450 2050 1450 1750
-Wire Wire Line
-	1250 2050 1450 2050
+	2150 2250 2150 2150
+Connection ~ 2150 2250
+Wire Wire Line
+	1950 2250 2150 2250
+Wire Wire Line
+	2150 2150 2150 2050
+Connection ~ 2150 2150
+Wire Wire Line
+	1950 2150 2150 2150
+Wire Wire Line
+	2150 2050 2150 1950
+Connection ~ 2150 2050
+Wire Wire Line
+	1950 2050 2150 2050
+Connection ~ 2150 1950
+Wire Wire Line
+	2150 2350 2150 2250
+Wire Wire Line
+	1950 2350 2150 2350
+Wire Wire Line
+	1300 2350 1300 2250
+Connection ~ 1300 2350
+Wire Wire Line
+	1450 2350 1300 2350
+Wire Wire Line
+	1300 2250 1300 2150
+Connection ~ 1300 2250
+Wire Wire Line
+	1450 2250 1300 2250
+Wire Wire Line
+	1300 2150 1300 2050
+Connection ~ 1300 2150
+Wire Wire Line
+	1450 2150 1300 2150
+Wire Wire Line
+	1300 2050 1300 1950
+Connection ~ 1300 2050
+Wire Wire Line
+	1450 2050 1300 2050
+Wire Wire Line
+	1300 1950 1450 1950
+Wire Wire Line
+	1300 2650 1300 2350
+Wire Wire Line
+	2150 1950 2150 1650
+Wire Wire Line
+	1950 1950 2150 1950
 $Comp
 L power:+5V #PWR0136
 U 1 1 5DFAB11E
-P 1450 1750
-F 0 "#PWR0136" H 1450 1600 50  0001 C CNN
-F 1 "+5V" H 1465 1923 50  0000 C CNN
-F 2 "" H 1450 1750 50  0001 C CNN
-F 3 "" H 1450 1750 50  0001 C CNN
-	1    1450 1750
+P 2150 1650
+F 0 "#PWR0136" H 2150 1500 50  0001 C CNN
+F 1 "+5V" H 2165 1823 50  0000 C CNN
+F 2 "" H 2150 1650 50  0001 C CNN
+F 3 "" H 2150 1650 50  0001 C CNN
+	1    2150 1650
 	-1   0    0    -1
 $EndComp
@@
 L power:GND #PWR0135
 U 1 1 5DFAAD3F
-P 600 2750
-F 0 "#PWR0135" H 600 2500 50  0001 C CNN
-F 1 "GND" H 605 2577 50  0000 C CNN
-F 2 "" H 600 2750 50  0001 C CNN
-F 3 "" H 600 2750 50  0001 C CNN
-	1    600  2750
+P 1300 2650
+F 0 "#PWR0135" H 1300 2400 50  0001 C CNN
+F 1 "GND" H 1305 2477 50  0000 C CNN
+F 2 "" H 1300 2650 50  0001 C CNN
+F 3 "" H 1300 2650 50  0001 C CNN
+	1    1300 2650
 	1    0    0    -1
 $EndComp
@@
 L Connector_Generic:Conn_02x05_Odd_Even J8
 U 1 1 5DFA830C
-P 950 2250
-F 0 "J8" H 1000 2700 50  0000 C CNN
-F 1 "Conn_02x05_Odd_Even" H 1000 2600 50  0000 C CNN
-F 2 "Connector_PinHeader_2.54mm:PinHeader_2x05_P2.54mm_Vertical" H 950 2250 50  0001 C CNN
-F 3 "~" H 950 2250 50  0001 C CNN
-	1    950  2250
-	1    0    0    -1
-$EndComp
-$Comp
-L Connector_Generic:Conn_01x02 J1
-U 1 1 5DA4A282
-P 1900 2100
-F 0 "J1" H 1800 1850 50  0000 C CNN
-F 1 "Conn_01x02" H 1800 2250 50  0001 C CNN
-F 2 "Connector_PinHeader_2.54mm:PinHeader_1x02_P2.54mm_Vertical" H 1900 2100 50  0001 C CNN
-F 3 "~" H 1900 2100 50  0001 C CNN
-	1    1900 2100
-	-1   0    0    1
-$EndComp
-Wire Wire Line
-	2100 2100 2650 2100
-Text Notes 1400 1500 0    50   ~ 0
+P 1650 2150
+F 0 "J8" H 1700 2600 50  0000 C CNN
+F 1 "Conn_02x05_Odd_Even" H 1700 2500 50  0000 C CNN
+F 2 "Connector_PinHeader_2.54mm:PinHeader_2x05_P2.54mm_Vertical" H 1650 2150 50  0001 C CNN
+F 3 "~" H 1650 2150 50  0001 C CNN
+	1    1650 2150
+	1    0    0    -1
+$EndComp
+Text Notes 2100 1400 0    50   ~ 0
 5V
-Text Notes 2050 2450 2    50   ~ 0
+Text Notes 2050 2600 2    50   ~ 0
 add legends
 Wire Wire Line
@@
 	3150 1900 3150 2000
 Wire Wire Line
-	2100 2000 3150 2000
-Wire Wire Line
 	3250 2750 3250 2850
 Wire Wire Line
@@
 	3150 2750 3150 2850
 Wire Wire Line
-	2650 2850 3150 2850
+	2900 2850 3150 2850
 $Comp
 L Connector:Screw_Terminal_01x02 J4
@@
 	0    1    -1   0
 $EndComp
-Text Notes 1450 7000 0    50   ~ 0
+Text Notes 3500 5500 0    50   ~ 0
 Use case: To program RL78 uC, use this economic programmer.\nDownload free Renases Flash Programmer (Free)\nRenesas & RL78 are registerred trademarks of Renesas.\nAll other trademarks are owned by respective owners.\nDesigned using KiCAD - open souced PCB design tool.\n
+Text Label 2750 2000 0    50   ~ 0
+TL
+Wire Wire Line
+	2700 2000 3150 2000
+Wire Wire Line
+	2700 2100 2900 2100
+$Comp
+L Connector_Generic:Conn_01x02 J1
+U 1 1 5DA4A282
+P 2500 2100
+F 0 "J1" H 2400 1850 50  0000 C CNN
+F 1 "Conn_01x02" H 2400 2250 50  0001 C CNN
+F 2 "Connector_PinHeader_2.54mm:PinHeader_1x02_P2.54mm_Vertical" H 2500 2100 50  0001 C CNN
+F 3 "~" H 2500 2100 50  0001 C CNN
+	1    2500 2100
+	-1   0    0    1
+$EndComp
 $EndSCHEMATC
